File: V3s/DevBoardV1/Schematics/V3s_DevBoard_V1.sch (KiCad schematic (older format))
At the start: 49 parts, among them U4 BBQ10KBD

Commit message: Further progress
Parts:
- added R? (x3): 75, symbol Device:R_Small
- added U?: ADV7123, symbol V3s:ADV7123
- added U?: VGA, symbol V3s:VGA
Connections:
- net VSS: now also R?.1, R?.1, R?.1, U?.1 (G0), U?.14 (B0), U?.15 (B1), U?.2 (G1), U?.39 (R0), U?.40 (R1)
- net VSync: now reaches U?.34 (PE3)
- net VSync: now also U?.14 (VSync)
- net HSync: now reaches U?.35 (PE2)
- net HSync: now also U?.13 (HSync)
- new net: R?.2, U?.28 (IOB), U?.3 (B)
- new net: R?.2, U?.2 (G), U?.32 (IOG)
- new net: R?.2, U?.1 (R), U?.34 (IOR)
Other:
- moved on the sheet: C?, J?, R?, U?, Y?
